Commit message: ubuntu22 调试通了moveit2 gazebo联动

File: dock_robot_ws/src/dock_robot_description/urdf/dock_robot.ros2_control.xacro (robot description, xacro)
@@ -2,5 +2,5 @@
 <robot xmlns:xacro="http://www.ros.org/wiki/xacro">
     <xacro:macro name="my_robot_ros2_control" params="name initial_positions_file">
-        <xacro:property name="initial_positions" value="${xacro.load_yaml(initial_positions_file)['initial_positions']}"/>
+        <xacro:property name="initial_positions" value="${xacro.xacro.load_yaml(initial_positions_file)['initial_positions']}"/>
         <ros2_control name="${name}" type="system">
             <hardware>

File: dock_robot_ws/src/dock_robot_moveit_config/config/my_robot.ros2_control.xacro (robot description, xacro)
@@ -2,5 +2,5 @@
 <robot xmlns:xacro="http://www.ros.org/wiki/xacro">
     <xacro:macro name="my_robot_ros2_control" params="name initial_positions_file">
-        <xacro:property name="initial_positions" value="${load_yaml(initial_positions_file)['initial_positions']}"/>
+        <xacro:property name="initial_positions" value="${xacro.load_yaml(initial_positions_file)['initial_positions']}"/>
         <ros2_control name="${name}" type="system">
             <hardware>

Commit message: 重新生成arm的DH模型，gazebo中目前有抖动的现象，需要解决

File: dock_robot_ws/src/dock_robot_description/urdf/dock_robot.ros2_control.xacro (robot description, xacro)
@@ -2,5 +2,5 @@
 <robot xmlns:xacro="http://www.ros.org/wiki/xacro">
     <xacro:macro name="my_robot_ros2_control" params="name initial_positions_file">
-        <xacro:property name="initial_positions" value="${xacro.xacro.load_yaml(initial_positions_file)['initial_positions']}"/>
+        <xacro:property name="initial_positions" value="${xacro.load_yaml(initial_positions_file)['initial_positions']}"/>
         <ros2_control name="${name}" type="system">
             <hardware>
@@ -49,41 +49,41 @@
                 <state_interface name="velocity"/>
             </joint>
-            <joint name="jointR1">
+            <joint name="jointr1">
                 <command_interface name="position"/>
                 <command_interface name="velocity"/>
                 <state_interface name="position">
-                  <param name="initial_value">${initial_positions['jointR1']}</param>
+                  <param name="initial_value">${initial_positions['jointr1']}</param>
                 </state_interface>
                 <state_interface name="velocity"/>
             </joint>
-            <joint name="jointR2">
+            <joint name="jointr2">
                 <command_interface name="position"/>
                 <command_interface name="velocity"/>
                 <state_interface name="position">
-                  <param name="initial_value">${initial_positions['jointR2']}</param>
+                  <param name="initial_value">${initial_positions['jointr2']}</param>
                 </state_interface>
                 <state_interface name="velocity"/>
             </joint>
-            <joint name="jointR3">
+            <joint name="jointr3">
                 <command_interface name="position"/>
                 <command_interface name="velocity"/>
                 <state_interface name="position">
-                  <param name="initial_value">${initial_positions['jointR3']}</param>
+                  <param name="initial_value">${initial_positions['jointr3']}</param>
                 </state_interface>
                 <state_interface name="velocity"/>
             </joint>
-            <joint name="jointR4">
+            <joint name="jointr4">
                 <command_interface name="position"/>
                 <command_interface name="velocity"/>
                 <state_interface name="position">
-                  <param name="initial_value">${initial_positions['jointR4']}</param>
+                  <param name="initial_value">${initial_positions['jointr4']}</param>
                 </state_interface>
                 <state_interface name="velocity"/>
             </joint>
-            <joint name="jointR5">
+            <joint name="jointr5">
                 <command_interface name="position"/>
                 <command_interface name="velocity"/>
                 <state_interface name="position">
-                  <param name="initial_value">${initial_positions['jointR5']}</param>
+                  <param name="initial_value">${initial_positions['jointr5']}</param>
                 </state_interface>
                 <state_interface name="velocity"/>

File: dock_robot_ws/src/dock_robot_description/urdf/left_arm.urdf (robot description, URDF)
Before this commit: robot None, 6 links, 5 joints
Links:
- removed link Link1
- removed link Link2
- removed link Link3
- removed link Link4
- removed link Link5
- added link link1, mass 0.038594; collision mesh filename=package://dock_robot_description/meshes/link1.STL; visual mesh filename=package://dock_robot_description/meshes/link1.STL
- added link link2, mass 0.053858; collision mesh filename=package://dock_robot_description/meshes/link2.STL; visual mesh filename=package://dock_robot_description/meshes/link2.STL
- added link link3, mass 0.048598; collision mesh filename=package://dock_robot_description/meshes/link3.STL; visual mesh filename=package://dock_robot_description/meshes/link3.STL
- added link link4, mass 0.10134; collision mesh filename=package://dock_robot_description/meshes/link4.STL; visual mesh filename=package://dock_robot_description/meshes/link4.STL
- added link link5, mass 0.24266; collision mesh filename=package://dock_robot_description/meshes/link5.STL; visual mesh filename=package://dock_robot_description/meshes/link5.STL
- link arm_base_link: geometry collision mesh filename=package://dock_robot_description/meshes/base_link.STL; visual mesh filename=package://dock_robot_description/meshes/base_link.STL
Joints:
- joint joint1: axis -1 0 0 -> 0 0 1; child Link1 -> link1; limit lower=-3.14 upper=3.14 effort=100 velocity=100 -> lower=${j1_min} upper=${j1_max} effort=2 velocity=3.14; origin xyz=0.041 0.00071917 0.0010978 rpy=0 0 0 -> xyz=0 0 0.07035 rpy=0 0 0
- joint joint2: axis 0 0 -1 -> 0 0 1; child Link2 -> link2; limit lower=-3.14 upper=3.14 effort=100 velocity=100 -> lower=${j2_min} upper=${j2_max} effort=1 velocity=3.14; origin xyz=0.0925 0 0.002 rpy=0 0 0 -> xyz=-0.00071917 -0.032448 0.06315 rpy=-1.5708 0 0; parent Link1 -> link1
- joint joint3: axis -0.99999 0.0041222 0 -> 0 0 1; child Link3 -> link3; limit lower=-3.14 upper=3.14 effort=100 velocity=100 -> lower=${j3_min} upper=${j3_max} effort=2 velocity=3.14; origin xyz=0.1061 -0.00043737 -0.002 rpy=0 0 0 -> xyz=0.0005866 -0.1423 0.03135 rpy=1.5708 0 0; parent Link2 -> link2
- joint joint4: axis -4.8622E-05 -0.011795 -0.99993 -> 0 0 1; child Link4 -> link4; limit lower=-3.14 upper=3.14 effort=100 velocity=100 -> lower=${j4_min} upper=${j4_max} effort=2 velocity=3.14; origin xyz=0.1535 -0.00071297 -0.0067995 rpy=0 0 0 -> xyz=0.00013677 -0.029398 0.1173 rpy=1.5708 0 -3.1416; parent Link3 -> link3
- joint joint5: axis 0.99996 -0.0092582 6.0584E-05 -> 0 0 1; child Link5 -> link5; limit lower=-3.14 upper=3.14 effort=100 velocity=100 -> lower=${j5_min} upper=${j5_max} effort=2 velocity=3.14; origin xyz=0.23199 -0.0020901 0.0049137 rpy=0 0 0 -> xyz=-0.002724 0.25434 0.031282 rpy=1.5708 0 3.1416; parent Link4 -> link4

File: dock_robot_ws/src/dock_robot_description/urdf/mobile_base.xacro (robot description, xacro)
@@ -210,10 +210,10 @@
         <parent link="head_link" />
         <child link="left_arm_link" />
-        <origin xyz="0 0.05 0.05" rpy=" 0 0 ${pi/2}" />
+        <origin xyz="0 0.05 0.05" rpy=" ${-pi/2} ${pi/2} 0" />
     </joint>
     <joint name="head_right_arm_joint" type="fixed">
         <parent link="head_link" />
         <child link="right_arm_link" />
-        <origin xyz="0 -0.05 0.05" rpy="0 0 ${-pi/2}" />
+        <origin xyz="0 -0.05 0.05" rpy="${pi/2} ${-pi/2} 0" />
     </joint>
 </robot>

File: dock_robot_ws/src/dock_robot_description/urdf/mobile_base_gazebo.xacro (robot description, xacro)
@@ -31,9 +31,9 @@
             <joint_name>joint4</joint_name>
             <joint_name>joint5</joint_name>
-            <joint_name>jointR1</joint_name>
-            <joint_name>jointR2</joint_name>
-            <joint_name>jointR3</joint_name>
-            <joint_name>jointR4</joint_name>
-            <joint_name>jointR5</joint_name>
+            <joint_name>jointr1</joint_name>
+            <joint_name>jointr2</joint_name>
+            <joint_name>jointr3</joint_name>
+            <joint_name>jointr4</joint_name>
+            <joint_name>jointr5</joint_name>
         </plugin>
     </gazebo>

File: dock_robot_ws/src/dock_robot_description/urdf/right_arm.urdf (robot description, URDF)
Before this commit: robot None, 6 links, 5 joints
Links:
- removed link Link1R
- removed link Link2R
- removed link Link3R
- removed link Link4R
- removed link Link5R
- added link linkr1, mass 0.038594; collision mesh filename=package://dock_robot_description/meshes/linkr1.STL; visual mesh filename=package://dock_robot_description/meshes/linkr1.STL
- added link linkr2, mass 0.053858; collision mesh filename=package://dock_robot_description/meshes/linkr2.STL; visual mesh filename=package://dock_robot_description/meshes/linkr2.STL
- added link linkr3, mass 0.048598; collision mesh filename=package://dock_robot_description/meshes/linkr3.STL; visual mesh filename=package://dock_robot_description/meshes/linkr3.STL
- added link linkr4, mass 0.10134; collision mesh filename=package://dock_robot_description/meshes/linkr4.STL; visual mesh filename=package://dock_robot_description/meshes/linkr4.STL
- added link linkr5, mass 0.24266; collision mesh filename=package://dock_robot_description/meshes/linkr5.STL; visual mesh filename=package://dock_robot_description/meshes/linkr5.STL
- link right_arm_base_link: geometry collision mesh filename=package://dock_robot_description/meshes/base_linkr.STL; visual mesh filename=package://dock_robot_description/meshes/base_linkr.STL
Joints:
- removed joint jointR1
- removed joint jointR2
- removed joint jointR3
- removed joint jointR4
- removed joint jointR5
- added joint jointr1: type revolute, parent right_arm_base_link, child linkr1, origin xyz=0 0 0.07035 rpy=0 0 0, axis 0 0 1, limit lower=${j1_min} upper=${j1_max} effort=2 velocity=3.14
- added joint jointr2: type revolute, parent linkr1, child linkr2, origin xyz=-0.00071917 -0.032448 0.06315 rpy=-1.5708 0 0, axis 0 0 1, limit lower=${j2_min} upper=${j2_max} effort=1 velocity=3.14
- added joint jointr3: type revolute, parent linkr2, child linkr3, origin xyz=0.0005866 -0.1423 0.03135 rpy=1.5708 0 0, axis 0 0 1, limit lower=${j3_min} upper=${j3_max} effort=2 velocity=3.14
- added joint jointr4: type revolute, parent linkr3, child linkr4, origin xyz=0.00013677 -0.029398 0.1173 rpy=1.5708 0 -3.1416, axis 0 0 1, limit lower=${j4_min} upper=${j4_max} effort=2 velocity=3.14
- added joint jointr5: type revolute, parent linkr4, child linkr5, origin xyz=-0.002724 0.25434 0.031282 rpy=1.5708 0 3.1416, axis 0 0 1, limit lower=${j5_min} upper=${j5_max} effort=2 velocity=3.14

File: dock_robot_ws/src/dock_robot_moveit_config/config/my_robot.gazebo.ros2_control.xacro (robot description, xacro)
@@ -44,36 +44,36 @@
                 <state_interface name="velocity"/>
             </joint>
-            <joint name="jointR1">
+            <joint name="jointr1">
                 <command_interface name="position"/>
                 <state_interface name="position">
-                  <param name="initial_value">${initial_positions['jointR1']}</param>
+                  <param name="initial_value">${initial_positions['jointr1']}</param>
                 </state_interface>
                 <state_interface name="velocity"/>
             </joint>
-            <joint name="jointR2">
+            <joint name="jointr2">
                 <command_interface name="position"/>
                 <state_interface name="position">
-                  <param name="initial_value">${initial_positions['jointR2']}</param>
+                  <param name="initial_value">${initial_positions['jointr2']}</param>
                 </state_interface>
                 <state_interface name="velocity"/>
             </joint>
-            <joint name="jointR3">
+            <joint name="jointr3">
                 <command_interface name="position"/>
                 <state_interface name="position">
-                  <param name="initial_value">${initial_positions['jointR3']}</param>
+                  <param name="initial_value">${initial_positions['jointr3']}</param>
                 </state_interface>
                 <state_interface name="velocity"/>
             </joint>
-            <joint name="jointR4">
+            <joint name="jointr4">
                 <command_interface name="position"/>
                 <state_interface name="position">
-                  <param name="initial_value">${initial_positions['jointR4']}</param>
+                  <param name="initial_value">${initial_positions['jointr4']}</param>
                 </state_interface>
                 <state_interface name="velocity"/>
             </joint>
-            <joint name="jointR5">
+            <joint name="jointr5">
                 <command_interface name="position"/>
                 <state_interface name="position">
-                  <param name="initial_value">${initial_positions['jointR5']}</param>
+                  <param name="initial_value">${initial_positions['jointr5']}</param>
                 </state_interface>
                 <state_interface name="velocity"/>

File: dock_robot_ws/src/dock_robot_moveit_config/config/my_robot.ros2_control.xacro (robot description, xacro)
@@ -44,36 +44,36 @@
                 <state_interface name="velocity"/>
             </joint>
-            <joint name="jointR1">
+            <joint name="jointr1">
                 <command_interface name="position"/>
                 <state_interface name="position">
-                  <param name="initial_value">${initial_positions['jointR1']}</param>
+                  <param name="initial_value">${initial_positions['jointr1']}</param>
                 </state_interface>
                 <state_interface name="velocity"/>
             </joint>
-            <joint name="jointR2">
+            <joint name="jointr2">
                 <command_interface name="position"/>
                 <state_interface name="position">
-                  <param name="initial_value">${initial_positions['jointR2']}</param>
+                  <param name="initial_value">${initial_positions['jointr2']}</param>
                 </state_interface>
                 <state_interface name="velocity"/>
             </joint>
-            <joint name="jointR3">
+            <joint name="jointr3">
                 <command_interface name="position"/>
                 <state_interface name="position">
-                  <param name="initial_value">${initial_positions['jointR3']}</param>
+                  <param name="initial_value">${initial_positions['jointr3']}</param>
                 </state_interface>
                 <state_interface name="velocity"/>
             </joint>
-            <joint name="jointR4">
+            <joint name="jointr4">
                 <command_interface name="position"/>
                 <state_interface name="position">
-                  <param name="initial_value">${initial_positions['jointR4']}</param>
+                  <param name="initial_value">${initial_positions['jointr4']}</param>
                 </state_interface>
                 <state_interface name="velocity"/>
             </joint>
-            <joint name="jointR5">
+            <joint name="jointr5">
                 <command_interface name="position"/>
                 <state_interface name="position">
-                  <param name="initial_value">${initial_positions['jointR5']}</param>
+                  <param name="initial_value">${initial_positions['jointr5']}</param>
                 </state_interface>
                 <state_interface name="velocity"/>

File: dock_robot_ws/src/dock_robot_moveit_config/config/my_robot.urdf.xacro (robot description, xacro)
@@ -6,4 +6,4 @@
     <!-- Import control_xacro -->
     <xacro:include filename="my_robot.ros2_control.xacro" />
-    <xacro:my_robot_ros2_control name="FakeSystem2" initial_positions_file="$(arg initial_positions_file)"/>
+    <xacro:my_robot_ros2_control name="FakeSystem22" initial_positions_file="$(arg initial_positions_file)"/>
 </robot>

Commit message: 加入桥接文件，解决moveit中拖不动的问题

File: dock_robot_ws/src/dock_robot_description/urdf/dock_robot.ros2_control.xacro (robot description, xacro)
@@ -6,5 +6,6 @@
             <hardware>
                 <!-- By default, set up controllers for simulation. This won't work on real hardware -->
-                <plugin>mock_components/GenericSystem</plugin>
+                <!-- <plugin>mock_components/GenericSystem</plugin> -->
+                <plugin>gz_ros2_control/GazeboSimSystem</plugin>
                 <param name="calculate_dynamics">true</param>
             </hardware>

File: dock_robot_ws/src/dock_robot_description/urdf/mobile_base.xacro (robot description, xacro)
@@ -88,5 +88,5 @@
     </link>
     <link name="left_arm_link">
-        <!-- <origin xyz="0 0.05 0.05" rpy="0 0 0" /> -->
+        <!-- <origin xyz="0 0 -0.15" rpy="0 0 0" /> -->
     </link>
     <link name="right_arm_link" >
@@ -210,10 +210,10 @@
         <parent link="head_link" />
         <child link="left_arm_link" />
-        <origin xyz="0 0.05 0.05" rpy=" ${-pi/2} ${pi/2} 0" />
+        <origin xyz="0 0.03 0.05" rpy=" ${-pi/2} ${pi/2} 0" />
     </joint>
     <joint name="head_right_arm_joint" type="fixed">
         <parent link="head_link" />
         <child link="right_arm_link" />
-        <origin xyz="0 -0.05 0.05" rpy="${pi/2} ${-pi/2} 0" />
+        <origin xyz="0 -0.03 0.05" rpy="${pi/2} ${-pi/2} 0" />
     </joint>
 </robot>

File: dock_robot_ws/src/dock_robot_description/urdf/mobile_base_gazebo.xacro (robot description, xacro)
@@ -9,5 +9,5 @@
         <mu2 value="0.1" />
     </gazebo>
-    <gazebo>
+    <!-- <gazebo>
         <plugin filename="gz-sim-diff-drive-system" name="gz::sim::systems::DiffDrive" >
             <left_joint>base_left_wheel_joint</left_joint>
@@ -37,4 +37,4 @@
             <joint_name>jointr5</joint_name>
         </plugin>
-    </gazebo>
+    </gazebo> -->
 </robot>

File: dock_robot_ws/src/dock_robot_moveit_config/config/my_robot.gazebo.urdf.xacro (robot description, xacro)
@@ -4,7 +4,5 @@
     <!-- Import arm urdf file -->
     <xacro:include filename="$(find dock_robot_description)/urdf/dock_robot.urdf.xacro" />
-    <!--添加Gazebo所需的专有标签-->
     <gazebo>
-        <!--添加world-joint使机械臂固定在仿真场景中-->
         <!-- <joint name="world_joint" type="fixed">
             <parent>world</parent>
