Commit message: 添加left arm电机控制接口

File: dock_robot_ws/src/dock_robot_description/urdf/dock_robot.urdf.xacro (robot description, xacro)
@@ -9,5 +9,5 @@
     <xacro:include filename="left_arm.urdf" />
     <xacro:include filename="right_arm.urdf" />
-     <xacro:include filename="dock_robot.ros2_control.xacro" />
+     <!-- <xacro:include filename="dock_robot.ros2_control.xacro" /> -->
      <xacro:include filename="camera.urdf.xacro" />
      <xacro:include filename="imu.urdf.xacro" />

File: dock_robot_ws/src/dock_robot_description/urdf/left_arm.urdf (robot description, URDF)
Before this commit: robot None, 6 links, 5 joints
Joints:
- joint joint1: limit lower=${j1_min} upper=${j1_max} effort=2 velocity=3.14 -> lower=${j1_min} upper=${j1_max} effort=10 velocity=0.78
- joint joint2: limit lower=${j2_min} upper=${j2_max} effort=1 velocity=3.14 -> lower=${j2_min} upper=${j2_max} effort=10 velocity=0.78
- joint joint3: limit lower=${j3_min} upper=${j3_max} effort=2 velocity=3.14 -> lower=${j3_min} upper=${j3_max} effort=10 velocity=0.78
- joint joint4: limit lower=${j4_min} upper=${j4_max} effort=2 velocity=3.14 -> lower=${j4_min} upper=${j4_max} effort=10 velocity=0.78
- joint joint5: limit lower=${j5_min} upper=${j5_max} effort=2 velocity=3.14 -> lower=${j5_min} upper=${j5_max} effort=10 velocity=0.78

File: dock_robot_ws/src/dock_robot_description/urdf/right_arm.urdf (robot description, URDF)
Before this commit: robot arm, 6 links, 5 joints
Joints:
- joint jointr1: limit lower=${j1_min} upper=${j1_max} effort=2 velocity=3.14 -> lower=${j1_min} upper=${j1_max} effort=10 velocity=0.78
- joint jointr2: limit lower=${j2_min} upper=${j2_max} effort=1 velocity=3.14 -> lower=${j2_min} upper=${j2_max} effort=10 velocity=0.78
- joint jointr3: limit lower=${j3_min} upper=${j3_max} effort=2 velocity=3.14 -> lower=${j3_min} upper=${j3_max} effort=10 velocity=0.78
- joint jointr4: limit lower=${j4_min} upper=${j4_max} effort=2 velocity=3.14 -> lower=${j4_min} upper=${j4_max} effort=10 velocity=0.78
- joint jointr5: limit lower=${j5_min} upper=${j5_max} effort=2 velocity=3.14 -> lower=${j5_min} upper=${j5_max} effort=10 velocity=0.78

File: dock_robot_ws/src/dock_robot_moveit_config/config/my_robot.urdf.xacro (robot description, xacro)
@@ -6,4 +6,4 @@
     <!-- Import control_xacro -->
     <xacro:include filename="my_robot.ros2_control.xacro" />
-    <xacro:my_robot_ros2_control name="FakeSystem22" initial_positions_file="$(arg initial_positions_file)"/>
+    <xacro:my_robot_ros2_control name="DockSystem" initial_positions_file="$(arg initial_positions_file)"/>
 </robot>
