Commit message: 调整为右臂跟实际的硬件相对应

File: dock_robot_ws/src/dock_robot_description/urdf/right_arm.urdf (robot description, URDF)
Before this commit: robot arm, 6 links, 5 joints
Joints:
- joint jointr2: axis 0 0 1 -> 0 0 -1

File: dock_robot_ws/src/dock_robot_moveit_config/config/my_robot.ros2_control.xacro (robot description, xacro)
@@ -9,5 +9,40 @@
                 <param name="calculate_dynamics">true</param> -->
                 <plugin>arm_hardware/ArmHardwareInterface</plugin>
-              </hardware>
+            </hardware>
+            <joint name="jointr1">
+                <command_interface name="position"/>
+                <state_interface name="position">
+                  <param name="initial_value">${initial_positions['jointr1']}</param>
+                </state_interface>
+                <!-- <state_interface name="velocity"/> -->
+            </joint>
+            <joint name="jointr2">
+                <command_interface name="position"/>
+                <state_interface name="position">
+                  <param name="initial_value">${initial_positions['jointr2']}</param>
+                </state_interface>
+                <!-- <state_interface name="velocity"/> -->
+            </joint>
+            <joint name="jointr3">
+                <command_interface name="position"/>
+                <state_interface name="position">
+                  <param name="initial_value">${initial_positions['jointr3']}</param>
+                </state_interface>
+                <!-- <state_interface name="velocity"/> -->
+            </joint>
+            <joint name="jointr4">
+                <command_interface name="position"/>
+                <state_interface name="position">
+                  <param name="initial_value">${initial_positions['jointr4']}</param>
+                </state_interface>
+                <!-- <state_interface name="velocity"/> -->
+            </joint>
+            <joint name="jointr5">
+                <command_interface name="position"/>
+                <state_interface name="position">
+                  <param name="initial_value">${initial_positions['jointr5']}</param>
+                </state_interface>
+                <!-- <state_interface name="velocity"/> -->
+            </joint>
             <joint name="joint1">
                 <command_interface name="position"/>
@@ -45,39 +80,4 @@
                 <!-- <state_interface name="velocity"/> -->
             </joint>
-            <joint name="jointr1">
-                <command_interface name="position"/>
-                <state_interface name="position">
-                  <param name="initial_value">${initial_positions['jointr1']}</param>
-                </state_interface>
-                <!-- <state_interface name="velocity"/> -->
-            </joint>
-            <joint name="jointr2">
-                <command_interface name="position"/>
-                <state_interface name="position">
-                  <param name="initial_value">${initial_positions['jointr2']}</param>
-                </state_interface>
-                <!-- <state_interface name="velocity"/> -->
-            </joint>
-            <joint name="jointr3">
-                <command_interface name="position"/>
-                <state_interface name="position">
-                  <param name="initial_value">${initial_positions['jointr3']}</param>
-                </state_interface>
-                <!-- <state_interface name="velocity"/> -->
-            </joint>
-            <joint name="jointr4">
-                <command_interface name="position"/>
-                <state_interface name="position">
-                  <param name="initial_value">${initial_positions['jointr4']}</param>
-                </state_interface>
-                <!-- <state_interface name="velocity"/> -->
-            </joint>
-            <joint name="jointr5">
-                <command_interface name="position"/>
-                <state_interface name="position">
-                  <param name="initial_value">${initial_positions['jointr5']}</param>
-                </state_interface>
-                <!-- <state_interface name="velocity"/> -->
-            </joint>
             <joint name="base_left_wheel_joint">
                 <command_interface name="position"/>

Commit message: 修正电机运动与仿真里面运动方向一致

File: dock_robot_ws/src/dock_robot_description/urdf/right_arm.urdf (robot description, URDF)
Before this commit: robot arm, 6 links, 5 joints
Joints:
- joint jointr4: axis 0 0 1 -> 0 0 -1
