Commit message: gazebo 开发中

File: dock_robot_ws/src/dock_robot_description/urdf/common_properties.xacro (robot description, xacro)
@@ -17,3 +17,31 @@
     <xacro:property name="j5_min" value="-3.14" />
     <xacro:property name="j5_max" value="3.14" />
+     <xacro:macro name="box_inertia" params="m x y z o_xyz o_rpy">
+        <inertial>
+            <mass value="${m}" />
+                <origin xyz="${o_xyz}" rpy="${o_rpy}" />
+            <inertia ixx="${(m/12) * (y*y + z*z)}" ixy="0" ixz="0"
+                     iyy="${(m/12) * (x*x + z*z)}" iyz="0"
+                     izz="${(m/12) * (x*x + y*y)}" >
+            </inertia>
+        </inertial>
+    </xacro:macro>
+    <xacro:macro name="cylinder_inertia" params="m r l o_xyz o_rpy">
+        <inertial>
+            <mass value="${m}" />
+            <origin xyz="${o_xyz}" rpy="${o_rpy}" />
+            <inertia ixx="${(m/12) * (3*r*r + l*l)}" ixy="0" ixz="0"
+                     iyy="${(m/12) * (3*r*r + l*l)}" iyz="0"
+                     izz="${(m/2) * (r*r)}" />
+        </inertial>
+    </xacro:macro>
+    <xacro:macro name="sphere_inertia" params="m r o_xyz o_rpy">
+        <inertial>
+            <mass value="${m}" />
+            <origin xyz="${o_xyz}" rpy="${o_rpy}" />
+            <inertia ixx="${(2/5) * m * r * r}" ixy="0" ixz="0"
+                     iyy="${(2/5) * m * r * r}" iyz="0"
+                     izz="${(2/5) * m * r * r}" />
+        </inertial>
+    </xacro:macro>
 </robot>

File: dock_robot_ws/src/dock_robot_description/urdf/dock_robot.urdf.xacro (robot description, xacro)
@@ -4,4 +4,5 @@
     <xacro:include filename="common_properties.xacro" />
     <xacro:include filename="mobile_base.xacro" />
+    <xacro:include filename="mobile_base_gazebo.xacro" />
     <!-- <xacro:include filename="arm1.xacro" /> -->
     <!-- <xacro:include filename="gripper.xacro" /> -->

File: dock_robot_ws/src/dock_robot_description/urdf/left_arm.urdf (robot description, URDF)
Before this commit: robot None, 6 links, 5 joints
Links:
- link Link1: geometry collision mesh filename=package://dock_robot_description/meshes/Link1.stl; visual mesh filename=package://dock_robot_description/meshes/Link1.stl
- link Link2: geometry collision mesh filename=package://dock_robot_description/meshes/Link2.stl; visual mesh filename=package://dock_robot_description/meshes/Link2.stl
- link Link3: geometry collision mesh filename=package://dock_robot_description/meshes/Link3.stl; visual mesh filename=package://dock_robot_description/meshes/Link3.stl
- link Link4: geometry collision mesh filename=package://dock_robot_description/meshes/Link4.stl; visual mesh filename=package://dock_robot_description/meshes/Link4.stl
- link Link5: geometry collision mesh filename=package://dock_robot_description/meshes/Link5.stl; visual mesh filename=package://dock_robot_description/meshes/Link5.stl
- link arm_base_link: geometry collision mesh filename=package://dock_robot_description/meshes/arm_base_link.stl; visual mesh filename=package://dock_robot_description/meshes/arm_base_link.stl

File: dock_robot_ws/src/dock_robot_description/urdf/mobile_base.xacro (robot description, xacro)
@@ -34,4 +34,6 @@
             <origin xyz="0 0 ${base_height/2}" rpy="0 0 0" />
         </collision>
+        <xacro:box_inertia m="5.0" x="${base_length}" y="${base_width}" z="${base_height}"
+                            o_xyz="0 0 ${base_height/2}" o_rpy="0 0 0" />
     </link>
     <link name="lift_link">
@@ -49,4 +51,6 @@
             <origin xyz="0 0 ${lift_height/2}" rpy="0 0 0" />
         </collision>
+        <xacro:box_inertia m="2.0" x="${lift_length}" y="${lift_width}" z="${lift_height}"
+                            o_xyz="0 0 ${lift_height/2}" o_rpy="0 0 0" />
     </link>
     <link name="controller_link">
@@ -64,4 +68,6 @@
             <origin xyz="0 0 ${controller_height/2}" rpy="0 0 0" />
         </collision>
+        <xacro:box_inertia m="2.0" x="${controller_length}" y="${controller_width}" z="${controller_height}"
+                            o_xyz="0 0 ${controller_height/2}" o_rpy="0 0 0" />
     </link>
     <link name="head_link">
@@ -79,4 +85,5 @@
             <origin xyz="0 0 ${head_length/2}" rpy="0 0 0" />
         </collision>
+        <xacro:cylinder_inertia m="0.5" r="${head_radius}" l="${head_length}" o_xyz="0 0 ${head_length/2}" o_rpy="0 0 0" />
     </link>
     <link name="left_arm_link">
@@ -100,4 +107,6 @@
             <origin xyz="0 0 0" rpy="${pi/2.0} 0 0" />
         </collision>
+        <xacro:cylinder_inertia m="1.0" r="${wheel_radius}" l="${wheel_length}"
+                                    o_xyz="0 0 0" o_rpy="${pi / 2.0} 0 0" />
     </link>
     <link name="left_wheel_link">
@@ -115,4 +124,6 @@
             <origin xyz="0 0 0" rpy="${pi/2.0} 0 0" />
         </collision>
+        <xacro:cylinder_inertia m="1.0" r="${wheel_radius}" l="${wheel_length}"
+                                    o_xyz="0 0 0" o_rpy="${pi / 2.0} 0 0" />
     </link>
     <link name ="left_caster_wheel_link">
@@ -131,4 +142,5 @@
             <material name="grey" />
         </collision>
+        <xacro:sphere_inertia m="0.5" r="${caster_wheel_length}" o_xyz="0 0 0" o_rpy="0 0 0" />
     </link>
     <link name ="right_caster_wheel_link">
@@ -147,4 +159,5 @@
             <material name="grey" />
         </collision>
+        <xacro:sphere_inertia m="0.5" r="${caster_wheel_length}" o_xyz="0 0 0" o_rpy="0 0 0" />
     </link>
     <joint name="base_joint" type="fixed">

File: dock_robot_ws/src/dock_robot_description/urdf/right_arm.urdf (robot description, URDF)
Before this commit: robot None, 6 links, 5 joints
Links:
- link Link1R: geometry collision mesh filename=package://dock_robot_description/meshes/Link1R.stl; visual mesh filename=package://dock_robot_description/meshes/Link1R.stl
- link Link2R: geometry collision mesh filename=package://dock_robot_description/meshes/Link2R.stl; visual mesh filename=package://dock_robot_description/meshes/Link2R.stl
- link Link3R: geometry collision mesh filename=package://dock_robot_description/meshes/Link3R.stl; visual mesh filename=package://dock_robot_description/meshes/Link3R.stl
- link Link4R: geometry collision mesh filename=package://dock_robot_description/meshes/Link4R.stl; visual mesh filename=package://dock_robot_description/meshes/Link4R.stl
- link Link5R: geometry collision mesh filename=package://dock_robot_description/meshes/Link5R.stl; visual mesh filename=package://dock_robot_description/meshes/Link5R.stl

Commit message: 调通setPoseTarget程序

File: dock_robot_ws/src/dock_robot_description/urdf/common_properties.xacro (robot description, xacro)
@@ -17,5 +17,5 @@
     <xacro:property name="j5_min" value="-3.14" />
     <xacro:property name="j5_max" value="3.14" />
-     <xacro:macro name="box_inertia" params="m x y z o_xyz o_rpy">
+    <xacro:macro name="box_inertia" params="m x y z o_xyz o_rpy">
         <inertial>
             <mass value="${m}" />

Commit message: 添加Lidar、Camera模型

File: dock_robot_ws/src/dock_robot_description/urdf/common_properties.xacro (robot description, xacro)
@@ -6,4 +6,10 @@
     <material name="grey">
         <color rgba="0.5 0.5 0.5 1" />
+    </material>
+    <material name="yellow">
+        <color rgba="1.0 1.0 0.0 1.0"/>
+    </material>
+    <material name="orange">
+        <color rgba="1.0 0.5 0.0 1.0"/>
     </material>
     <xacro:property name="j1_min" value="-1.57" />

File: dock_robot_ws/src/dock_robot_description/urdf/dock_robot.urdf.xacro (robot description, xacro)
@@ -10,4 +10,8 @@
     <xacro:include filename="right_arm.urdf" />
      <xacro:include filename="dock_robot.ros2_control.xacro" />
+     <xacro:include filename="camera.urdf.xacro" />
+     <xacro:include filename="imu.urdf.xacro" />
+     <xacro:include filename="laser.urdf.xacro" />
+     <xacro:include filename="sensor_gazebo.xacro" />
      <!-- <xacro:my_robot_ros2_control name="FakeSystem" initial_positions_file="$(arg initial_positions_file)"/> -->
      <!-- <joint name="gripper_base_joint" type="fixed">
@@ -26,3 +30,6 @@
         <origin xyz="0 0 0" rpy="0 0 0" />
     </joint>
+    <xacro:laser_xacro xyz="0.0 0.0 0.1" />
+    <xacro:camera_xacro xyz="0.0 0.0 0.02" />
+    <!-- <xacro:imu_xacro xyz="0.0 0.0 0.02" /> -->
 </robot>

Commit message: 添加IMU

File: dock_robot_ws/src/dock_robot_description/urdf/common_properties.xacro (robot description, xacro)
@@ -2,5 +2,5 @@
 <robot xmlns:xacro="http://www.ros.org/wiki/xacro">
     <material name="green">
-        <color rgba="0 0.5 0 1" />
+        <color rgba="0 0.5 0 0.8" />
     </material>
     <material name="grey">

File: dock_robot_ws/src/dock_robot_description/urdf/dock_robot.urdf.xacro (robot description, xacro)
@@ -30,6 +30,6 @@
         <origin xyz="0 0 0" rpy="0 0 0" />
     </joint>
-    <xacro:laser_xacro xyz="0.0 0.0 0.1" />
+    <xacro:laser_xacro xyz="0.1615 0.0 0.212" />
     <xacro:camera_xacro xyz="0.0 0.0 0.02" />
-    <!-- <xacro:imu_xacro xyz="0.0 0.0 0.02" /> -->
+    <xacro:imu_xacro xyz="0.0 0.0 0.081" />
 </robot>

File: dock_robot_ws/src/dock_robot_description/urdf/laser.urdf.xacro (robot description, xacro)
@@ -47,5 +47,6 @@
         </joint>
         <joint name="laser_cylinder_joint" type="fixed">
-            <parent link="head_link"/>
+            <!-- <parent link="head_link"/> -->
+            <parent link="base_link"/>
             <child link="laser_cylinder_link"/>
             <origin xyz="${xyz}" rpy="0.0 0.0 0.0"/>

File: dock_robot_ws/src/dock_robot_description/urdf/sensor_gazebo.xacro (robot description, xacro)
@@ -10,4 +10,26 @@
             <child_frame_id>base_footprint</child_frame_id>`
         </plugin>
+    </gazebo> -->
+    <!-- <gazebo reference="base_left_wheel_joint, base_right_wheel_joint">
+        <plugin name='gz::sim::systems::DiffDrive' filename='gz-sim-diff-drive-system'>
+        <left_joint>base_left_wheel_joint</left_joint>
+        <right_joint>base_right_wheel_joint</right_joint>
+        <wheel_separation>0.1615</wheel_separation>
+        <wheel_radius>0.1</wheel_radius>
+        <max_linear_acceleration>1</max_linear_acceleration>
+        <min_linear_acceleration>-1</min_linear_acceleration>
+        <max_angular_acceleration>2</max_angular_acceleration>
+        <min_angular_acceleration>-2</min_angular_acceleration>
+        <max_linear_velocity>0.46</max_linear_velocity>
+        <min_linear_velocity>-0.46</min_linear_velocity>
+        <max_angular_velocity>1.9</max_angular_velocity>
+        <min_angular_velocity>-1.9</min_angular_velocity>
+        <topic>/cmd_vel</topic>
+        <odom_topic>/odom</odom_topic>
+        <tf_topic>/tf</tf_topic>
+        <frame_id>odom</frame_id>
+        <child_frame_id>base_footprint</child_frame_id>
+        <odom_publish_frequency>30</odom_publish_frequency>
+      </plugin>
     </gazebo> -->
     <!-- <gazebo>
@@ -79,4 +101,16 @@
         </sensor>
     </gazebo>
+    <gazebo reference="imu_link">
+        <sensor name="imu_sensor" type="imu">
+          <always_on>1</always_on>
+          <update_rate>100</update_rate>
+          <visualize>true</visualize>
+          <topic>imu</topic>
+          <frame_id>imu_link</frame_id>
+          <gz_frame_id>imu_link</gz_frame_id>
+          <ignition_frame_id>imu_link</ignition_frame_id>
+          <ros_frame_id>imu_link</ros_frame_id>
+        </sensor>
+    </gazebo>
     <!-- </sensor> -->
     <!-- 在 sensor 标签结束后添加 -->

Commit message: 精细化小车模型，更改srdf文件

File: dock_robot_ws/src/dock_robot_description/urdf/common_properties.xacro (robot description, xacro)
@@ -2,8 +2,8 @@
 <robot xmlns:xacro="http://www.ros.org/wiki/xacro">
     <material name="green">
-        <color rgba="0 0.5 0 0.8" />
+        <color rgba="0 0.5 0 1.0" />
     </material>
     <material name="grey">
-        <color rgba="0.5 0.5 0.5 1" />
+        <color rgba="0.5 0.5 0.5 1.0" />
     </material>
     <material name="yellow">

File: dock_robot_ws/src/dock_robot_description/urdf/dock_robot.urdf.xacro (robot description, xacro)
@@ -3,6 +3,13 @@
     <xacro:arg name="initial_positions_file" default="initial_positions.yaml" />
     <xacro:include filename="common_properties.xacro" />
-    <xacro:include filename="mobile_base.xacro" />
-    <xacro:include filename="mobile_base_gazebo.xacro" />
+   <!-- 底盘类型参数 -->
+    <xacro:arg name="base_type" default="wheeltec"/>
+    <xacro:if value="$(eval base_type == 'mobile')">
+        <xacro:include filename="mobile_base.xacro"/>
+        <xacro:include filename="mobile_base_gazebo.xacro"/>
+    </xacro:if>
+    <xacro:if value="$(eval base_type == 'wheeltec')">
+        <xacro:include filename="S100_diff_robot_with_body.urdf.xacro"/>
+    </xacro:if>
     <!-- <xacro:include filename="arm1.xacro" /> -->
     <!-- <xacro:include filename="gripper.xacro" /> -->
@@ -10,8 +17,8 @@
     <xacro:include filename="right_arm.urdf" />
      <!-- <xacro:include filename="dock_robot.ros2_control.xacro" /> -->
-     <xacro:include filename="camera.urdf.xacro" />
+     <!-- <xacro:include filename="camera.urdf.xacro" />
      <xacro:include filename="imu.urdf.xacro" />
      <xacro:include filename="laser.urdf.xacro" />
-     <xacro:include filename="sensor_gazebo.xacro" />
+     <xacro:include filename="sensor_gazebo.xacro" /> -->
      <!-- <xacro:my_robot_ros2_control name="FakeSystem" initial_positions_file="$(arg initial_positions_file)"/> -->
      <!-- <joint name="gripper_base_joint" type="fixed">
@@ -30,7 +37,7 @@
         <origin xyz="0 0 0" rpy="0 0 0" />
     </joint>
-    <xacro:laser_xacro xyz="0.1615 0.0 0.212" />
+    <!-- <xacro:laser_xacro xyz="0.1615 0.0 0.212" />
     <xacro:camera_xacro xyz="0.0 0.0 0.02" />
-    <xacro:imu_xacro xyz="0.0 0.0 0.0" />
+    <xacro:imu_xacro xyz="0.0 0.0 0.0" /> -->
     <!-- <xacro:imu_xacro xyz="0.0 0.0 0.081" /> -->
 </robot>

File: dock_robot_ws/src/dock_robot_moveit_config/config/my_robot.ros2_control.xacro (robot description, xacro)
@@ -80,5 +80,5 @@
                 <!-- <state_interface name="velocity"/> -->
             </joint>
-            <joint name="base_left_wheel_joint">
+            <joint name="lf_wheel_joint">
                 <command_interface name="position"/>
                 <state_interface name="position">
@@ -87,5 +87,5 @@
                 <!-- <state_interface name="velocity"/> -->
             </joint>
-            <joint name="base_right_wheel_joint">
+            <joint name="rf_wheel_joint">
                 <command_interface name="position"/>
                 <state_interface name="position">

Commit message: 调试mtc_pick_place

File: dock_robot_ws/src/dock_robot_description/urdf/common_properties.xacro (robot description, xacro)
@@ -11,4 +11,7 @@
     </material>
     <material name="orange">
+        <color rgba="1.0 0.5 0.0 1.0"/>
+    </material>
+    <material name="dark_green">
         <color rgba="1.0 0.5 0.0 1.0"/>
     </material>

File: dock_robot_ws/src/dock_robot_description/urdf/dock_robot.urdf.xacro (robot description, xacro)
@@ -13,5 +13,5 @@
     </xacro:if>
     <!-- <xacro:include filename="arm1.xacro" /> -->
-    <!-- <xacro:include filename="gripper.xacro" /> -->
+    <xacro:include filename="gripper.xacro" />
     <xacro:include filename="left_arm.urdf" />
     <xacro:include filename="right_arm.urdf" />
@@ -22,9 +22,9 @@
      <xacro:include filename="sensor_gazebo.xacro" /> -->
      <!-- <xacro:my_robot_ros2_control name="FakeSystem" initial_positions_file="$(arg initial_positions_file)"/> -->
-     <!-- <joint name="gripper_base_joint" type="fixed">
-        <parent link="left_arm_link" />
+    <joint name="gripper_base_joint" type="fixed">
+        <parent link="link5" />
         <child link="gripper_base_link" />
-        <origin xyz="0 0 0" rpy="-1.57 0 0" />
-    </joint> -->
+        <origin xyz="0 0 0" rpy="0 0 1.57" />
+    </joint>
     <joint name="left_arm_joint" type="fixed">
         <parent link="left_arm_link" />
