Commit message: 添加夹爪控制器，使用xyz进行模拟抓取

File: dock_robot_ws/src/dock_robot_description/urdf/gripper.xacro (robot description, xacro)
@@ -61,3 +61,9 @@
         <limit effort="1000.0" velocity="1.0" lower="-0.06" upper="0.0" />
     </joint>
+    <link name="left_gripper_tcp"/>
+    <joint name="left_gripper_tcp_joint" type="fixed">
+        <parent link="gripper_base_link"/>
+        <child link="left_gripper_tcp"/>
+        <origin xyz="0 0 0.04" rpy="1.5708 0 0"/>
+    </joint>
 </robot>

File: dock_robot_ws/src/dock_robot_moveit_config/config/my_robot.ros2_control.xacro (robot description, xacro)
@@ -101,4 +101,10 @@
                 <!-- <state_interface name="velocity"/> -->
             </joint>
+            <joint name="gripper_left_finger_joint">
+                <command_interface name="position"/>
+                <state_interface name="position">
+                  <param name="initial_value">${initial_positions['gripper_left_finger_joint']}</param>
+                </state_interface>
+            </joint>
         </ros2_control>
     </xacro:macro>
