Commit message: 调试左臂程序

File: dock_robot_ws/src/dock_robot_description/urdf/left_arm.urdf (robot description, URDF)
Before this commit: robot None, 6 links, 5 joints
Joints:
- joint joint2: axis 0 0 1 -> 0 0 -1
- joint joint4: axis 0 0 1 -> 0 0 -1

Commit message: 更改CAN参数修正电机方向

File: dock_robot_ws/src/dock_robot_description/urdf/left_arm.urdf (robot description, URDF)
Before this commit: robot None, 6 links, 5 joints
Joints:
- joint joint2: axis 0 0 -1 -> 0 0 1
- joint joint4: axis 0 0 -1 -> 0 0 1

File: dock_robot_ws/src/dock_robot_description/urdf/right_arm.urdf (robot description, URDF)
Before this commit: robot arm, 6 links, 5 joints
Joints:
- joint jointr2: axis 0 0 -1 -> 0 0 1
- joint jointr4: axis 0 0 -1 -> 0 0 1

Commit message: 硬件调试抓瓶子的动作

File: dock_robot_ws/src/dock_robot_description/urdf/left_arm.urdf (robot description, URDF)
Before this commit: robot None, 6 links, 5 joints
Joints:
- joint joint2: axis 0 0 1 -> 0 0 -1
- joint joint4: axis 0 0 1 -> 0 0 -1

File: dock_robot_ws/src/dock_robot_description/urdf/right_arm.urdf (robot description, URDF)
Before this commit: robot arm, 6 links, 5 joints
Joints:
- joint jointr2: axis 0 0 1 -> 0 0 -1
- joint jointr4: axis 0 0 1 -> 0 0 -1

File: dock_robot_ws/src/dock_robot_moveit_config/config/my_robot.ros2_control.xacro (robot description, xacro)
@@ -6,7 +6,7 @@
             <hardware>
                 <!-- By default, set up controllers for simulation. This won't work on real hardware -->
-                <plugin>mock_components/GenericSystem</plugin>
-                <param name="calculate_dynamics">true</param>
-                <!-- <plugin>arm_hardware/ArmHardwareInterface</plugin> -->
+                <!-- <plugin>mock_components/GenericSystem</plugin> -->
+                <!-- <param name="calculate_dynamics">true</param> -->
+                <plugin>arm_hardware/ArmHardwareInterface</plugin>
             </hardware>
             <joint name="joint1">
