Commit message: 增加left_arm相关程序

File: dock_robot_ws/src/dock_robot_moveit_config/config/my_robot.ros2_control.xacro (robot description, xacro)
@@ -10,4 +10,39 @@
                 <plugin>arm_hardware/ArmHardwareInterface</plugin>
             </hardware>
+            <joint name="joint1">
+                <command_interface name="position"/>
+                <state_interface name="position">
+                  <param name="initial_value">${initial_positions['joint1']}</param>
+                </state_interface>
+                <!-- <state_interface name="velocity"/> -->
+            </joint>
+            <joint name="joint2">
+                <command_interface name="position"/>
+                <state_interface name="position">
+                  <param name="initial_value">${initial_positions['joint2']}</param>
+                </state_interface>
+                <!-- <state_interface name="velocity"/> -->
+            </joint>
+            <joint name="joint3">
+                <command_interface name="position"/>
+                <state_interface name="position">
+                  <param name="initial_value">${initial_positions['joint3']}</param>
+                </state_interface>
+                <!-- <state_interface name="velocity"/> -->
+            </joint>
+            <joint name="joint4">
+                <command_interface name="position"/>
+                <state_interface name="position">
+                  <param name="initial_value">${initial_positions['joint4']}</param>
+                </state_interface>
+                <!-- <state_interface name="velocity"/> -->
+            </joint>
+            <joint name="joint5">
+                <command_interface name="position"/>
+                <state_interface name="position">
+                  <param name="initial_value">${initial_positions['joint5']}</param>
+                </state_interface>
+                <!-- <state_interface name="velocity"/> -->
+            </joint>
             <joint name="jointr1">
                 <command_interface name="position"/>
@@ -45,39 +80,4 @@
                 <!-- <state_interface name="velocity"/> -->
             </joint>
-            <joint name="joint1">
-                <command_interface name="position"/>
-                <state_interface name="position">
-                  <param name="initial_value">${initial_positions['joint1']}</param>
-                </state_interface>
-                <!-- <state_interface name="velocity"/> -->
-            </joint>
-            <joint name="joint2">
-                <command_interface name="position"/>
-                <state_interface name="position">
-                  <param name="initial_value">${initial_positions['joint2']}</param>
-                </state_interface>
-                <!-- <state_interface name="velocity"/> -->
-            </joint>
-            <joint name="joint3">
-                <command_interface name="position"/>
-                <state_interface name="position">
-                  <param name="initial_value">${initial_positions['joint3']}</param>
-                </state_interface>
-                <!-- <state_interface name="velocity"/> -->
-            </joint>
-            <joint name="joint4">
-                <command_interface name="position"/>
-                <state_interface name="position">
-                  <param name="initial_value">${initial_positions['joint4']}</param>
-                </state_interface>
-                <!-- <state_interface name="velocity"/> -->
-            </joint>
-            <joint name="joint5">
-                <command_interface name="position"/>
-                <state_interface name="position">
-                  <param name="initial_value">${initial_positions['joint5']}</param>
-                </state_interface>
-                <!-- <state_interface name="velocity"/> -->
-            </joint>
             <joint name="base_left_wheel_joint">
                 <command_interface name="position"/>

Commit message: 增加夹爪的ros2_control控制程序

File: dock_robot_ws/src/dock_robot_moveit_config/config/my_robot.ros2_control.xacro (robot description, xacro)
@@ -101,10 +101,10 @@
                 <!-- <state_interface name="velocity"/> -->
             </joint>
-            <joint name="gripper_left_finger_joint">
+            <!-- <joint name="gripper_left_finger_joint">
                 <command_interface name="position"/>
                 <state_interface name="position">
                   <param name="initial_value">${initial_positions['gripper_left_finger_joint']}</param>
                 </state_interface>
-            </joint>
+            </joint> -->
         </ros2_control>
     </xacro:macro>

File: dock_robot_ws/src/dock_robot_moveit_config/config/my_robot.urdf.xacro (robot description, xacro)
@@ -2,4 +2,8 @@
 <robot xmlns:xacro="http://www.ros.org/wiki/xacro" name="my_robot">
     <xacro:arg name="initial_positions_file" default="initial_positions.yaml" />
+    <xacro:arg name="gripper_serial_port" default="/dev/ttyACM0" />
+    <xacro:arg name="gripper_baudrate" default="115200" />
+    <xacro:arg name="gripper_speed" default="80" />
+    <xacro:arg name="gripper_initial_position" default="0.0" />
     <!-- Import my_robot urdf file -->
     <xacro:include filename="$(find dock_robot_description)/urdf/dock_robot.urdf.xacro" />
@@ -7,3 +11,10 @@
     <xacro:include filename="my_robot.ros2_control.xacro" />
     <xacro:my_robot_ros2_control name="DockSystem" initial_positions_file="$(arg initial_positions_file)"/>
+    <xacro:include filename="$(find dock_robot_gripper_hardware)/config/gripper_ros2_control.xacro" />
+    <xacro:gripper_ros2_control
+        name="GripperSystem"
+        serial_port="$(arg gripper_serial_port)"
+        baudrate="$(arg gripper_baudrate)"
+        speed="$(arg gripper_speed)"
+        initial_position="$(arg gripper_initial_position)"/>
 </robot>
